Commit message: created a ur3e_rg2_description package

File: Traj_Control/ur3e_moveit_config/config/ur3e.urdf (robot description, URDF)
Before this commit: robot ur, 13 links, 12 joints
Links:
- added link onrobot_base_link
- added link onrobot_finger_width_mock_link
- added link onrobot_gripper_tcp
- added link onrobot_left_finger_tip
- added link onrobot_left_inner_finger
- added link onrobot_left_inner_knuckle
- added link onrobot_left_outer_knuckle
- added link onrobot_right_finger_tip
- added link onrobot_right_inner_finger
- added link onrobot_right_inner_knuckle
- added link onrobot_right_outer_knuckle
Joints:
- added joint onrobot_finger_joint: type revolute, parent onrobot_base_link, child onrobot_left_outer_knuckle, origin xyz=0 -0.017178 0.125797 rpy=0 0 0, axis -1 0 0, limit lower=-0.558505 upper=0.785398 effort=1000 velocity=100, mimic joint=onrobot_finger_width multiplier=‑3.8343 offset=0.785398
- added joint onrobot_finger_width: type prismatic, parent onrobot_base_link, child onrobot_finger_width_mock_link, origin xyz=0 0 0 rpy=0 0 0, axis 0 0 1, limit lower=0 upper=0.110 effort=40 velocity=0.127
- added joint onrobot_left_finger_tip_joint: type fixed, parent onrobot_left_inner_finger, child onrobot_left_finger_tip, origin xyz=0 0.019 0.038 rpy=0 0 0
- added joint onrobot_left_inner_finger_joint: type revolute, parent onrobot_left_outer_knuckle, child onrobot_left_inner_finger, origin xyz=0 -0.039592 0.038177 rpy=0 0 0, axis 1 0 0, limit lower=-0.872665 upper=0.872665 effort=1000 velocity=100, mimic joint=onrobot_finger_joint multiplier=1
- added joint onrobot_left_inner_knuckle_joint: type revolute, parent onrobot_left_outer_knuckle, child onrobot_left_inner_knuckle, origin xyz=0 -0.007678 0.142297 rpy=0 0 0, axis 1 0 0, limit lower=-0.785398 upper=0.785398 effort=1000 velocity=100, mimic joint=onrobot_finger_joint multiplier=-1
- added joint onrobot_right_finger_tip_joint: type fixed, parent onrobot_right_inner_finger, child onrobot_right_finger_tip, origin xyz=0 -0.019 0.038 rpy=0 0 0
- added joint onrobot_right_inner_finger_joint: type revolute, parent onrobot_right_outer_knuckle, child onrobot_right_inner_finger, origin xyz=0 0.039592 0.038177 rpy=0 0 0, axis 1 0 0, limit lower=-0.872665 upper=0.872665 effort=1000 velocity=100, mimic joint=onrobot_finger_joint multiplier=1
- added joint onrobot_right_inner_knuckle_joint: type revolute, parent onrobot_right_outer_knuckle, child onrobot_right_inner_knuckle, origin xyz=0 0.007678 0.142297 rpy=0 0 0, axis 1 0 0, limit lower=-0.785398 upper=0.785398 effort=1000 velocity=100, mimic joint=onrobot_finger_joint multiplier=-1
- added joint onrobot_right_outer_knuckle_joint: type revolute, parent onrobot_base_link, child onrobot_right_outer_knuckle, origin xyz=0 0.017178 0.125797 rpy=0 0 3.14159265359, axis 1 0 0, limit lower=-0.785398 upper=0.785398 effort=1000 velocity=100, mimic joint=onrobot_finger_joint multiplier=-1
- added joint onrobot_tcp_joint: type fixed, parent onrobot_base_link, child onrobot_gripper_tcp, origin xyz=0 0 0.218 rpy=0 0 0
- added joint tool0-to-onrobot_base_link: type fixed, parent tool0, child onrobot_base_link, origin xyz=0 0 0.218 rpy=0 0 0
