Commit message: moveit package created

File: Traj_Control/ur3e_rg2_description/urdf/ur3e_rg2.urdf.xacro (robot description, xacro)
@@ -4,5 +4,5 @@
   <xacro:arg name="ur_type" default="ur3e"/>
   <xacro:arg name="onrobot_type" default="rg2"/>
-  <xacro:arg name="prefix" default=""/>
+  <xacro:arg name="prefix" default="ur3e_"/>
   <xacro:arg name="joint_limits_parameters_file" default="$(find ur_description)/config/$(arg ur_type)/joint_limits.yaml"/>
   <xacro:arg name="kinematics_parameters_file" default="$(find ur_description)/config/$(arg ur_type)/default_kinematics.yaml"/>
@@ -14,4 +14,6 @@
     parent="world"
     ur_type="$(arg ur_type)"
+    onrobot_type="$(arg onrobot_type)"
+    prefix="$(arg prefix)"
     joint_limits_parameters_file="$(arg joint_limits_parameters_file)"
     kinematics_parameters_file="$(arg kinematics_parameters_file)"

File: Traj_Control/ur3e_rg2_description/urdf/ur3e_rg2_macro.xacro (robot description, xacro)
@@ -3,20 +3,20 @@
   <xacro:include filename="$(find ur_description)/urdf/ur_macro.xacro"/>
   <xacro:include filename="$(find onrobot_description)/urdf/onrobot_macro.xacro"/>
-  <xacro:onrobot onrobot_type="$(arg onrobot_type)" prefix="$(arg prefix)"/>
   <xacro:macro name="ur3e_rg2" params="
     parent
     *origin
     ur_type
+    onrobot_type
+    prefix
     joint_limits_parameters_file
     kinematics_parameters_file
     physical_parameters_file
-    visual_parameters_file
-    ">
-  <joint name="$(arg prefix)onrobot_base_link_joint" type="fixed">
-    <origin xyz="0 0 0" rpy="0 0 0"/>
-    <parent link="$(arg prefix)tool0"/>
-    <child link="$(arg prefix)onrobot_base_link"/>
-  </joint>
-    <!--This will create the specific robot-->
+    visual_parameters_file">
+    <xacro:onrobot onrobot_type="${onrobot_type}" prefix="${prefix}"/>
+    <joint name="${prefix}onrobot_base_link_joint" type="fixed">
+      <origin xyz="0 0 0" rpy="0 0 0"/>
+      <parent link="${prefix}tool0"/>
+      <child link="${prefix}onrobot_base_link"/>
+    </joint>
     <xacro:ur_robot
       name="${ur_type}"
