Commit message: I like to moveit moveit

File: Traj_Control/ur3e_rg2_control/urdf/ur3e_rg2_controlled.urdf.xacro (robot description, xacro)
@@ -10,5 +10,5 @@
   <xacro:arg name="ur_type" default="ur3e"/>
   <xacro:arg name="onrobot_type" default="rg2"/>
-  <xacro:arg name="prefix" default="ur3e_"/>
+  <xacro:arg name="prefix" default=""/>
   <xacro:arg name="joint_limit_params" default="$(find ur3e_rg2_control)/config/$(arg ur_type)/joint_limits.yaml"/>
   <xacro:arg name="kinematics_params" default="$(find ur3e_rg2_control)/config/$(arg ur_type)/default_kinematics.yaml"/>
@@ -36,4 +36,5 @@
     physical_parameters_file="$(arg physical_params)"
     visual_parameters_file="$(arg visual_params)"
+    use_fake_hardware="$(arg use_fake_hardware)"
   >
     <origin xyz="0 0 1" rpy="0 0 0" />
@@ -41,5 +42,5 @@
   <!--Create the control tag for the UR robot-->
   <xacro:ur_ros2_control
-    name="$(arg ur_type)"
+    name="ur"
     tf_prefix="$(arg ur_type)_"
     hash_kinematics="${kinematics_hash}"
@@ -52,13 +53,4 @@
     headless_mode="$(arg headless_mode)"
   />
-  <!--Create the control tag for the Onrobot RG2 robot-->
-  <ros2_control name="onrobot_gripper" type="system">
-    <!-- You may need to update joint name depending on your gripper's setup -->
-    <joint name="$(arg prefix)gripper_joint">
-      <command_interface name="position"/>
-      <state_interface name="position"/>
-      <state_interface name="velocity"/>
-    </joint>
-  </ros2_control>
   <!--If you had more controlled devices in your description, e.g. a gripper, you can add another ros2_control tag here-->
 </robot>

File: Traj_Control/ur3e_rg2_description/urdf/ur3e_rg2.urdf.xacro (robot description, xacro)
@@ -4,5 +4,6 @@
   <xacro:arg name="ur_type" default="ur3e"/>
   <xacro:arg name="onrobot_type" default="rg2"/>
-  <xacro:arg name="prefix" default="ur3e_"/>
+  <xacro:arg name="prefix" default=""/>
+  <xacro:arg name="use_fake_hardware" default="false"/>
   <xacro:arg name="joint_limits_parameters_file" default="$(find ur_description)/config/$(arg ur_type)/joint_limits.yaml"/>
   <xacro:arg name="kinematics_parameters_file" default="$(find ur_description)/config/$(arg ur_type)/default_kinematics.yaml"/>
@@ -20,4 +21,5 @@
     physical_parameters_file="$(arg physical_parameters_file)"
     visual_parameters_file="$(arg visual_parameters_file)"
+    use_fake_hardware="$(arg use_fake_hardware)"
     >
       <origin xyz="0 0 1" rpy="0 0 0" />

File: Traj_Control/ur3e_rg2_description/urdf/ur3e_rg2_macro.xacro (robot description, xacro)
@@ -12,14 +12,18 @@
     kinematics_parameters_file
     physical_parameters_file
-    visual_parameters_file">
-    <xacro:onrobot onrobot_type="${onrobot_type}" prefix="${prefix}"/>
+    visual_parameters_file
+    use_fake_hardware">
+    <xacro:onrobot
+      onrobot_type="${onrobot_type}"
+      prefix="${prefix}"
+      use_fake_hardware="${use_fake_hardware}"/>
     <joint name="${prefix}onrobot_base_link_joint" type="fixed">
       <origin xyz="0 0 0" rpy="0 0 0"/>
-      <parent link="${prefix}tool0"/>
+      <parent link="tool0"/>
       <child link="${prefix}onrobot_base_link"/>
     </joint>
     <xacro:ur_robot
       name="${ur_type}"
-      tf_prefix="${ur_type}_"
+      tf_prefix=""
       parent="world"
       joint_limits_parameters_file="${joint_limits_parameters_file}"
@@ -27,4 +31,5 @@
       physical_parameters_file="${physical_parameters_file}"
       visual_parameters_file="${visual_parameters_file}"
+      use_fake_hardware="${use_fake_hardware}"
     >
       <origin xyz="0 0 0" rpy="0 0 0" />
