Commit message: Added new main which reads from topics and sends to the robot

File: Traj_Control/ur3e_rg2_moveit_config/srdf/ur_onrobot_macro.srdf.xacro (robot description, xacro)
@@ -31,5 +31,5 @@
     <!--GROUP STATES - Purpose - Define a named state for a particular group, in terms of joint values. This is useful to define states like 'folded arms'-->
     <group_state name="closed" group="${prefix}${name}_gripper">
-      <joint name="finger_width" value="0.049"/>
+      <joint name="finger_width" value="0.047"/>
     </group_state>
     <group_state name="open" group="${prefix}${name}_gripper">
